File: skematik/7-Juli-2026/skematik-monitor/adxl345.kicad_sch (KiCad schematic)
At the start: 2 parts, among them U1 DS18B20

Commit message: Update 3-Sep-2026
Parts:
- removed R1: R, symbol Device:R
- removed U1: DS18B20, Package_TO_SOT_THT:TO-92_Inline, symbol Sensor_Temperature:DS18B20
- added U7: ADXL345, Package_LGA:LGA-14_3x5mm_P0.8mm_LayoutBorder1x6y, symbol Sensor_Motion:ADXL343
Connections:
- net 3V3: now also U7.1 (Vdd_I/O)
- net GND: now also U7.2 (GND), U7.4 (GND), U7.5 (GND)
- new net SCL: U7.14 (SCL/SCLK)
- new net SDA: U7.13 (SDA/SDI/SDIO)
Other:
- note added: "Sensor Akselerometer"
