File: skematik/7-Juli-2026/skematik-monitor/skematik-monitor.kicad_pcb (KiCad board)
At the start: 2 copper layers, 66.5 x 76.1 mm, 6 parts, among them U1 ESP32-DevKitC, U4 ADXL345

Commit message: Security update
Other:
- board size 66.5 x 76.1 mm -> 48.5 x 76.1 mm
Changed lines of the file:
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@@
 	)
 	(gr_rect
-		(start 136.739847 50.910958)
-		(end 203.2 127)
+		(start 141.769923 49)
+		(end 190.230076 125.089042)
 		(stroke
 			(width 0.05)

Commit message: Update 3-Sep-2026
Routing:
- net SCL: track 40.2 -> 46.1 mm
- net SDA: track 45.7 -> 49.8 mm
- net GPIO34: track 17.9 -> 14.9 mm
- net GND: track 48.8 -> 50.0 mm
Changed lines of the file:
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@@
 		(tenting front back)
 		(pcbplotparams
-			(layerselection 0x00000000_00000000_55555555_5755f5ff)
-			(plot_on_all_layers_selection 0x00000000_00000000_00000000_00000000)
+			(layerselection 0x00000000_00000000_55555555_d5557773)
+			(plot_on_all_layers_selection 0x00000000_00000000_00000000_00002003)
 			(disableapertmacros no)
 			(usegerberextensions no)
@@
 			(crossoutdnponfab yes)
 			(subtractmaskfromsilk no)
-			(outputformat 1)
+			(outputformat 4)
 			(mirror no)
-			(drillshape 1)
+			(drillshape 0)
 			(scaleselection 1)
 			(outputdirectory "")
@@
 	)
 	(segment
-		(start 182.720421 75.59928)
-		(end 183.428484 75.59928)
-		(width 0.2)
+		(start 151.38141 101.972206)
+		(end 151.38141 86.830445)
+		(width 0.5)
 		(layer "F.Cu")
 		(net 1)
 	)
 	(segment
-		(start 151.38141 101.972206)
-		(end 151.38141 86.830445)
-		(width 0.2)
+		(start 180.59928 75.59928)
+		(end 183.428484 75.59928)
+		(width 0.5)
 		(layer "F.Cu")
 		(net 1)
@@
 		(start 151.231888 78.851321)
 		(end 151.231888 86.680923)
-		(width 0.2)
+		(width 0.5)
 		(layer "F.Cu")
 		(net 1)
@@
 	(segment
 		(start 172.132476 64.536336)
-		(end 172.132476 65.011335)
-		(width 0.2)
+		(end 172.132476 67.132476)
+		(width 0.5)
 		(layer "F.Cu")
 		(net 1)
@@
 	)
 	(segment
-		(start 172.132476 65.011335)
-		(end 182.720421 75.59928)
-		(width 0.2)
+		(start 172.132476 67.132476)
+		(end 180.59928 75.59928)
+		(width 0.5)
 		(layer "F.Cu")
 		(net 1)
@@
 		(start 158.028484 108.61928)
 		(end 151.38141 101.972206)
-		(width 0.2)
+		(width 0.5)
 		(layer "F.Cu")
 		(net 1)
@@
 		(start 148.691888 78.851321)
 		(end 148.691888 75.748802)
-		(width 0.2)
+		(width 0.5)
 		(layer "F.Cu")
 		(net 2)
@@
 		(start 148.88141 97.758793)
 		(end 148.88141 86.830445)
-		(width 0.2)
+		(width 0.5)
 		(layer "F.Cu")
 		(net 2)
@@
 		(start 146.444092 100.196111)
 		(end 148.88141 97.758793)
-		(width 0.2)
+		(width 0.5)
 		(layer "F.Cu")
 		(net 2)
@@
 	)
 	(segment
-		(start 154.273979 102.141115)
-		(end 154.273979 89.513785)
+		(start 154 99)
+		(end 154.273979 98.726021)
 		(width 0.2)
 		(layer "F.Cu")
@@
 	)
 	(segment
+		(start 154.273979 98.726021)
+		(end 154.273979 89.513785)
+		(width 0.5)
+		(layer "F.Cu")
+		(net 3)
+	)
+	(segment
 		(start 154.273979 89.513785)
 		(end 158.028484 85.75928)
-		(width 0.2)
+		(width 0.5)
 		(layer "F.Cu")
 		(net 3)
 	)
 	(via
-		(at 154.273979 102.141115)
+		(at 154 99)
 		(size 3)
 		(drill 2)
@@
 		(start 156.589604 75.59928)
 		(end 151.38141 75.59928)
-		(width 0.2)
+		(width 0.5)
 		(layer "F.Cu")
 		(net 4)
@@
 		(start 162.009013 64.536336)
 		(end 158.028484 68.516865)
-		(width 0.2)
+		(width 0.5)
 		(layer "F.Cu")
 		(net 4)
@@
 		(start 158.028484 68.516865)
 		(end 158.028484 75.59928)
-		(width 0.2)
+		(width 0.5)
 		(layer "F.Cu")
 		(net 4)
@@
 		(start 168.932476 64.536336)
 		(end 162.009013 64.536336)
-		(width 0.2)
+		(width 0.5)
 		(layer "F.Cu")
 		(net 4)
 	)
 	(segment
-		(start 168.815508 63.536336)
-		(end 167.406701 62.127529)
-		(width 0.2)
+		(start 186 78.107764)
+		(end 183.428484 80.67928)
+		(width 0.5)
 		(layer "F.Cu")
 		(net 24)
 	)
 	(segment
-		(start 167.406701 56.688864)
-		(end 169.072122 56.688864)
-		(width 0.2)
+		(start 170.688864 56.688864)
+		(end 186 72)
+		(width 0.5)
 		(layer "F.Cu")
 		(net 24)
 	)
 	(segment
-		(start 184.729484 72.346226)
-		(end 184.729484 79.37828)
-		(width 0.2)
+		(start 168.932476 63.536336)
+		(end 165.536336 63.536336)
+		(width 0.5)
 		(layer "F.Cu")
 		(net 24)
 	)
 	(segment
-		(start 167.406701 62.127529)
+		(start 165 59.095565)
 		(end 167.406701 56.688864)
-		(width 0.2)
+		(width 0.5)
 		(layer "F.Cu")
 		(net 24)
 	)
 	(segment
-		(start 169.072122 56.688864)
-		(end 184.729484 72.346226)
-		(width 0.2)
+		(start 165.536336 63.536336)
+		(end 165 63)
+		(width 0.5)
 		(layer "F.Cu")
 		(net 24)
 	)
 	(segment
-		(start 184.729484 79.37828)
-		(end 183.428484 80.67928)
-		(width 0.2)
+		(start 186 72)
+		(end 186 78.107764)
+		(width 0.5)
 		(layer "F.Cu")
 		(net 24)
 	)
 	(segment
-		(start 168.932476 63.536336)
-		(end 168.815508 63.536336)
-		(width 0.2)
+		(start 167.406701 56.688864)
+		(end 169.072122 56.688864)
+		(width 0.5)
+		(layer "F.Cu")
+		(net 24)
+	)
+	(segment
+		(start 165 62.127529)
+		(end 165 59.095565)
+		(width 0.5)
 		(layer "F.Cu")
 		(net 24)
 	)
 	(segment
+		(start 169.072122 56.688864)
+		(end 170.688864 56.688864)
+		(width 0.5)
+		(layer "F.Cu")
+		(net 24)
+	)
+	(segment
+		(start 165 63)
+		(end 165 62.127529)
+		(width 0.5)
+		(layer "F.Cu")
+		(net 24)
+	)
+	(segment
+		(start 171.865241 53.865241)
+		(end 188 70)
+		(width 0.5)
+		(layer "F.Cu")
+		(net 35)
+	)
+	(segment
 		(start 168.932476 59.058025)
 		(end 169.04526 58.945241)
@@
 	)
 	(segment
-		(start 185.130484 69.950465)
-		(end 185.130484 86.59728)
-		(width 0.2)
+		(start 188 70)
+		(end 188 83.727764)
+		(width 0.5)
 		(layer "F.Cu")
 		(net 35)
 	)
 	(segment
-		(start 185.130484 86.59728)
-		(end 183.428484 88.29928)
-		(width 0.2)
+		(start 169.04526 53.865241)
+		(end 171.865241 53.865241)
+		(width 0.5)
 		(layer "F.Cu")
 		(net 35)
 	)
 	(segment
-		(start 168.932476 62.536336)
-		(end 168.932476 59.058025)
-		(width 0.2)
+		(start 188 83.727764)
+		(end 183.428484 88.29928)
+		(width 0.5)
 		(layer "F.Cu")
 		(net 35)
 	)
 	(segment
-		(start 169.04526 53.865241)
-		(end 185.130484 69.950465)
-		(width 0.2)
+		(start 168.932476 62.536336)
+		(end 168.932476 59.058025)
+		(width 0.5)
 		(layer "F.Cu")
 		(net 35)
